File: boards/30keys/Ghazal/Ghazal.kicad_pcb (KiCad board)
At the start: 2 copper layers, 262.4 x 124.1 mm, 107 parts, among them J2 Conn_01x03_Pin, J3 Conn_01x06, SW1 SW_Push, SW10 SW_Push, SW11 SW_Push, SW12 SW_Push, SW13 SW_Push, SW14 SW_Push, SW15 SW_Push, SW16 SW_Push, SW17 SW_Push, SW18 SW_Push, SW19 SW_Push, SW2 SW_Push, SW20 SW_Push, SW21 SW_Push, SW22 SW_Push, SW23 SW_Push, SW24 SW_Push, SW25 SW_SPDT, SW26 SW_Push, SW27 SW_Push, SW28 SW_Push, SW29 SW_Push, SW3 SW_Push, SW30 SW_Push, SW31 SW_Push, SW32 SW_Push, SW33 SW_Push, SW34 SW_Push, SW35 SW_Push, SW37 SW_Push, SW4 SW_Push, SW5 SW_Push, SW6 SW_Push, SW7 SW_Push, SW8 SW_Push, SW9 SW_Push, U1 nice_nano

Commit message: tmp
Parts:
- removed D39, D40, D41, D42, D43, D44, D45: 1N4148, Diode_SMD:D_SOD-123
- removed HAT1, HAT2: 5Way-Tactile_K1-1506DN-01, Alaa:5Way-non-reverse
- added D26: 1N4148, Diode_SMD:D_SOD-123, B.Cu at (94.5, 106.0)
- added D31: 1N4148, Diode_SMD:D_SOD-123, B.Cu at (192.4, 111.1)
- added D34: 1N4148, Diode_SMD:D_SOD-123, B.Cu at (50.8, 135.0)
- added SW20: SW_Push, Alaa:Kailh_hotswap_only_MX-CHOC, F.Cu at (64.2, 107.3)
- added SW27: SW_Push, Alaa:Kailh_hotswap_only_MX-CHOC, F.Cu at (102.8, 102.3)
- added SW32: SW_Push, Alaa:Kailh_hotswap_only_MX-CHOC, F.Cu at (197.4, 101.9)
- moved D36 35.2 mm to (50.8, 138.3), turned to 180 degrees
- moved D37 31.5 mm to (50.8, 141.7), turned to 180 degrees
- moved D38 29.7 mm to (50.8, 145.0), turned to 180 degrees
- moved H3 15.4 mm to (174.9, 110.6)
- moved H2 11.4 mm to (118.7, 111.1)
- moved D25 8.95 mm to (108.3, 70.0)
- moved SW26 8.27 mm to (117.3, 66.6)
- moved D31 8.22 mm to (185.3, 93.4)
- moved D32 8.22 mm to (178.1, 75.7)
- moved SW33 8.22 mm to (183.2, 66.5)
- moved SW32 8.22 mm to (190.3, 84.1)
- moved D26 8.08 mm to (101.3, 87.9)
- moved SW27 8.00 mm to (110.1, 84.4)
- moved JP6 1.72 mm to (126.7, 44.9)
- moved JP5 1.20 mm to (126.8, 39.8)
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Connections:
- D1 pad 2: col0 -> unconnected-(D1-A-Pad2)
- D10 pad 2: col1 -> unconnected-(D10-A-Pad2)
- D11 pad 2: col2 -> unconnected-(D11-A-Pad2)
- D12 pad 2: col3 -> unconnected-(D12-A-Pad2)
- D13 pad 2: col4 -> unconnected-(D13-A-Pad2)
- D14 pad 2: col5 -> unconnected-(D14-A-Pad2)
- D15 pad 2: col6 -> unconnected-(D15-A-Pad2)
- D16 pad 2: col7 -> unconnected-(D16-A-Pad2)
- D17 pad 2: col0 -> unconnected-(D17-A-Pad2)
- D18 pad 2: col1 -> unconnected-(D18-A-Pad2)
- D19 pad 2: col2 -> unconnected-(D19-A-Pad2)
- D2 pad 2: col1 -> unconnected-(D2-A-Pad2)
- D20 pad 2: col3 -> unconnected-(D20-A-Pad2)
- D21 pad 2: col4 -> unconnected-(D21-A-Pad2)
- D22 pad 2: col5 -> unconnected-(D22-A-Pad2)
- D23 pad 2: col6 -> unconnected-(D23-A-Pad2)
- D24 pad 2: col7 -> unconnected-(D24-A-Pad2)
- D25 pad 2: col0 -> unconnected-(D25-A-Pad2)
- D26 pad 2: col1 -> unconnected-(D26-A-Pad2)
- D27 pad 2: col2 -> unconnected-(D27-A-Pad2)
- D28 pad 2: col3 -> unconnected-(D28-A-Pad2)
- D29 pad 2: col4 -> unconnected-(D29-A-Pad2)
- D3 pad 2: col2 -> unconnected-(D3-A-Pad2)
- D30 pad 2: col5 -> unconnected-(D30-A-Pad2)
- D31 pad 2: col6 -> unconnected-(D31-A-Pad2)
- D32 pad 2: col7 -> unconnected-(D32-A-Pad2)
- D33 pad 2: col6 -> unconnected-(D33-A-Pad2)
- D35 pad 2: col7 -> unconnected-(D35-A-Pad2)
- D36 pad 2: col0 -> unconnected-(D36-A-Pad2)
- D37 pad 2: col1 -> unconnected-(D37-A-Pad2)
- D38 pad 2: col2 -> unconnected-(D38-A-Pad2)
- D4 pad 2: col3 -> unconnected-(D4-A-Pad2)
- D5 pad 2: col4 -> unconnected-(D5-A-Pad2)
- D6 pad 2: col5 -> unconnected-(D6-A-Pad2)
- D7 pad 2: col6 -> unconnected-(D7-A-Pad2)
- D8 pad 2: col7 -> unconnected-(D8-A-Pad2)
- D9 pad 2: col0 -> unconnected-(D9-A-Pad2)
- SW1 pad 1: row_0 -> unconnected-(SW1-Pad1)
- SW10 pad 1: row_1 -> unconnected-(SW10-Pad1)
- SW11 pad 1: row_1 -> unconnected-(SW11-Pad1)
- SW12 pad 1: row_1 -> unconnected-(SW12-Pad1)
- SW13 pad 1: row_1 -> unconnected-(SW13-Pad1)
- SW14 pad 1: row_1 -> unconnected-(SW14-Pad1)
- SW15 pad 1: row_1 -> unconnected-(SW15-Pad1)
- SW16 pad 1: row_1 -> unconnected-(SW16-Pad1)
- SW17 pad 1: row_2 -> unconnected-(SW17-Pad1)
- SW18 pad 1: row_2 -> unconnected-(SW18-Pad1)
- SW19 pad 1: row_2 -> unconnected-(SW19-Pad1)
- SW2 pad 1: row_0 -> unconnected-(SW2-Pad1)
- SW20 pad 1: row_2 -> unconnected-(SW20-Pad1)
- SW21 pad 1: row_2 -> unconnected-(SW21-Pad1)
- SW22 pad 1: row_2 -> unconnected-(SW22-Pad1)
- SW23 pad 1: row_2 -> unconnected-(SW23-Pad1)
- SW24 pad 1: row_2 -> unconnected-(SW24-Pad1)
- SW26 pad 1: row_3 -> unconnected-(SW26-Pad1)
- SW27 pad 1: row_3 -> unconnected-(SW27-Pad1)
- SW28 pad 1: row_3 -> unconnected-(SW28-Pad1)
- SW29 pad 1: row_3 -> unconnected-(SW29-Pad1)
- SW3 pad 1: row_0 -> unconnected-(SW3-Pad1)
- SW30 pad 1: row_3 -> unconnected-(SW30-Pad1)
- SW31 pad 1: row_3 -> unconnected-(SW31-Pad1)
- SW32 pad 1: row_3 -> unconnected-(SW32-Pad1)
- SW33 pad 1: row_3 -> unconnected-(SW33-Pad1)
- SW35 pad 1: row_4 -> unconnected-(SW35-Pad1)
- SW37 pad 1: row_4 -> unconnected-(SW37-Pad1)
- SW4 pad 1: row_0 -> unconnected-(SW4-Pad1)
- SW5 pad 1: row_0 -> unconnected-(SW5-Pad1)
- SW6 pad 1: row_0 -> unconnected-(SW6-Pad1)
- SW7 pad 1: row_0 -> unconnected-(SW7-Pad1)
- SW8 pad 1: row_0 -> unconnected-(SW8-Pad1)
- SW9 pad 1: row_1 -> unconnected-(SW9-Pad1)
Routing:
- net row_2: track 354.6 -> 0.00 mm, vias 12 -> 0
- net row_1: track 327.9 -> 0.00 mm, vias 9 -> 0
- net row_0: track 317.3 -> 0.00 mm, vias 8 -> 0
- net col3: track 314.2 -> 0.00 mm, vias 7 -> 0
- net col4: track 310.1 -> 0.00 mm, vias 6 -> 0
- net row_3: track 308.4 -> 0.00 mm, vias 8 -> 0
- net col6: track 269.8 -> 0.00 mm, vias 9 -> 0
- net col7: track 251.7 -> 0.00 mm, vias 7 -> 0
- net col0: track 231.0 -> 0.00 mm, vias 5 -> 0
- net row_4: track 214.5 -> 0.00 mm, vias 4 -> 0
- net col1: track 209.3 -> 0.00 mm, vias 3 -> 0
- net col2: track 205.9 -> 0.00 mm, vias 5 -> 0
- net col5: track 185.5 -> 0.00 mm, vias 5 -> 0
- net row_5: track 160.2 -> 0.00 mm, vias 3 -> 0
- net +3V3: track 108.9 -> 0.00 mm, vias 3 -> 0
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