File: boards/30keys/Ghazal/Ghazal.kicad_sch (KiCad schematic)
At the start: 105 parts, among them J2 Conn_01x03_Pin, J3 Conn_01x06, SW1 SW_Push, SW10 SW_Push, SW11 SW_Push, SW12 SW_Push, SW13 SW_Push, SW14 SW_Push, SW15 SW_Push, SW16 SW_Push, SW17 SW_Push, SW18 SW_Push, SW19 SW_Push, SW2 SW_Push, SW20 SW_Push, SW21 SW_Push, SW22 SW_Push, SW23 SW_Push, SW24 SW_Push, SW25 SW_SPDT, SW26 SW_Push, SW27 SW_Push, SW28 SW_Push, SW29 SW_Push, SW3 SW_Push, SW30 SW_Push, SW31 SW_Push, SW32 SW_Push, SW33 SW_Push, SW34 SW_Push, SW35 SW_Push, SW37 SW_Push, SW4 SW_Push, SW5 SW_Push, SW6 SW_Push, SW7 SW_Push, SW8 SW_Push, SW9 SW_Push, U4 nice_nano

Commit message: tmp
Parts:
- removed D36, D37, D38, D39, D40, D41, D42, D43, D44, D45: 1N4148, Diode_SMD:D_SOD-123, symbol Device:D
- removed HAT1, HAT2: 5Way-Tactile_K1-1506DN-01, Alaa:5Way-non-reverse, symbol DjinnSymbols:5Way-Tactile_K1-1506DN-01
- added D34, D36, D37, D38: 1N4148, Diode_SMD:D_SOD-123, symbol alaa:Diode_1N4148
- added SW36, SW38, SW39, SW40: SW_Push, Alaa:Kailh_hotswap_only_MX-CHOC, symbol Switch:SW_Push
Connections:
- net col0: no longer D1.2 (A), D17.2 (A), D25.2 (A), D9.2 (A)
- net col1: no longer D10.2 (A), D18.2 (A), D2.2 (A), D26.2 (A)
- net col2: no longer D11.2 (A), D19.2 (A), D27.2 (A), D3.2 (A)
- net col3: no longer D12.2 (A), D20.2 (A), D28.2 (A), D4.2 (A)
- net col4: no longer D13.2 (A), D21.2 (A), D29.2 (A), D5.2 (A)
- net col5: no longer D14.2 (A), D22.2 (A), D30.2 (A), D6.2 (A)
- net col6: no longer D15.2 (A), D23.2 (A), D31.2 (A), D33.2 (A), D7.2 (A)
- net col7: no longer D16.2 (A), D24.2 (A), D32.2 (A), D35.2 (A), D8.2 (A)
- net row_0: no longer SW1.1, SW2.1, SW3.1, SW4.1, SW5.1, SW6.1, SW7.1, SW8.1
- net row_1: no longer SW10.1, SW11.1, SW12.1, SW13.1, SW14.1, SW15.1, SW16.1, SW9.1
- net row_2: no longer SW17.1, SW18.1, SW19.1, SW20.1, SW21.1, SW22.1, SW23.1, SW24.1
- net row_3: no longer SW26.1, SW27.1, SW28.1, SW29.1, SW30.1, SW31.1, SW32.1, SW33.1
- net row_4: no longer SW35.1, SW37.1
- new net: D37.1 (K), SW39.2
- new net: D36.1 (K), SW38.2
- new net: D34.1 (K), SW36.2
- new net: D38.1 (K), SW40.2
Other:
- note removed: "5-Way Tactile D-Pad"
- moved on the sheet: D1, D10, D11, D12, D13, D15, D17, D18, D19, D2, D20, D21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
